Commit message: rover

File: robot_rover/urdf/ros2_control.urdf.xacro (robot description, xacro)
@@ -65,4 +65,22 @@
         <state_interface name="effort"/>
       </joint>
+      <joint name="03_arm_link1_part1_joint">
+        <state_interface name="effort"/>
+      </joint>
+      <joint name="04_arm_link2_part1_joint">
+        <state_interface name="effort"/>
+      </joint>
+      <joint name="05_arm_link3_T_joint">
+        <state_interface name="effort"/>
+      </joint>
+      <joint name="06_arm_base_fingers_R_joint">
+        <state_interface name="effort"/>
+      </joint>
+      <joint name="07_arm_finger_right_joint">
+        <state_interface name="effort"/>
+      </joint>
+      <joint name="08_arm_finger_left_joint">
+        <state_interface name="effort"/>
+      </joint>
     </ros2_control>
   </xacro:macro>
